File: warmingTray_v2/warmingTray_v2.kicad_pcb (KiCad board)
At the start: 2 copper layers, 116.1 x 53.8 mm, 38 parts, among them J1 Jack-DC, P1 Power, P2 Analog, P3 Analog, P4 Digital, P5 PWM, P6 PWM, P7 Communication

Commit message: Lots of controller changes
Parts:
- moved PAD5-1 1.15 mm to (129.4, 113.2)
- moved PAD1-1 1.14 mm to (139.7, 113.2)
Routing:
- net /2(**): track 38.1 -> 29.9 mm
- net /Pad8: track 79.6 -> 83.1 mm
- net /Pad7: track 64.9 -> 68.3 mm
- net /Pad6: track 50.5 -> 53.5 mm
- net /11(**): track 121.6 -> 124.0 mm
- net /12(**): track 129.5 -> 127.3 mm
- net /VCC5: track 243.8 -> 245.5 mm, vias 4 -> 3
- net /13(**): track 123.4 -> 124.8 mm
- net /Pad3: track 46.2 -> 47.3 mm
- net /Pad5: track 54.4 -> 55.4 mm
- net /32: track 19.2 -> 19.8 mm
- net /30: track 19.9 -> 20.5 mm
- net /28: track 19.5 -> 20.1 mm

Commit message: Large Update of all files
Parts:
- moved P4 43.2 mm to (211.5, 114.2), turned to 180 degrees
Changed lines of the file:
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@@
   )
   (footprint "Connector_PinHeader_2.54mm:PinHeader_2x18_P2.54mm_Vertical" (layer "F.Cu")
-    (at 208.28 71.12)
+    (at 211.455 114.173 180)
     (descr "Through hole straight pin header, 2x18, 2.54mm pitch, double rows")
     (tags "Through hole pin header THT 2x18 2.54mm double row")
@@
     (fp_line (start 3.81 44.45) (end -1.27 44.45)
       (stroke (width 0.1) (type solid)) (layer "F.Fab"))
-    (pad "1" thru_hole rect (at 0 0) (size 1.7 1.7) (drill 1) (layers "*.Cu" "*.Mask")
+    (pad "1" thru_hole rect (at 0 0 180) (size 1.7 1.7) (drill 1) (layers "*.Cu" "*.Mask")
       (net 2 "GND") (pinfunction "Pin_1") (pintype "passive"))
-    (pad "2" thru_hole oval (at 2.54 0) (size 1.7 1.7) (drill 1) (layers "*.Cu" "*.Mask")
+    (pad "2" thru_hole oval (at 2.54 0 180) (size 1.7 1.7) (drill 1) (layers "*.Cu" "*.Mask")
       (net 2 "GND") (pinfunction "Pin_2") (pintype "passive"))
-    (pad "3" thru_hole oval (at 0 2.54) (size 1.7 1.7) (drill 1) (layers "*.Cu" "*.Mask")
+    (pad "3" thru_hole oval (at 0 2.54 180) (size 1.7 1.7) (drill 1) (layers "*.Cu" "*.Mask")
       (net 45 "/52(SCK)") (pinfunction "Pin_3") (pintype "passive"))
-    (pad "4" thru_hole oval (at 2.54 2.54) (size 1.7 1.7) (drill 1) (layers "*.Cu" "*.Mask")
+    (pad "4" thru_hole oval (at 2.54 2.54 180) (size 1.7 1.7) (drill 1) (layers "*.Cu" "*.Mask")
       (net 46 "/53(SS)") (pinfunction "Pin_4") (pintype "passive"))
-    (pad "5" thru_hole oval (at 0 5.08) (size 1.7 1.7) (drill 1) (layers "*.Cu" "*.Mask")
+    (pad "5" thru_hole oval (at 0 5.08 180) (size 1.7 1.7) (drill 1) (layers "*.Cu" "*.Mask")
       (net 47 "/50") (pinfunction "Pin_5") (pintype "passive"))
-    (pad "6" thru_hole oval (at 2.54 5.08) (size 1.7 1.7) (drill 1) (layers "*.Cu" "*.Mask")
+    (pad "6" thru_hole oval (at 2.54 5.08 180) (size 1.7 1.7) (drill 1) (layers "*.Cu" "*.Mask")
       (net 48 "/51(MOSI)") (pinfunction "Pin_6") (pintype "passive"))
-    (pad "7" thru_hole oval (at 0 7.62) (size 1.7 1.7) (drill 1) (layers "*.Cu" "*.Mask")
+    (pad "7" thru_hole oval (at 0 7.62 180) (size 1.7 1.7) (drill 1) (layers "*.Cu" "*.Mask")
       (net 49 "/48") (pinfunction "Pin_7") (pintype "passive"))
-    (pad "8" thru_hole oval (at 2.54 7.62) (size 1.7 1.7) (drill 1) (layers "*.Cu" "*.Mask")
+    (pad "8" thru_hole oval (at 2.54 7.62 180) (size 1.7 1.7) (drill 1) (layers "*.Cu" "*.Mask")
       (net 50 "/49") (pinfunction "Pin_8") (pintype "passive"))
-    (pad "9" thru_hole oval (at 0 10.16) (size 1.7 1.7) (drill 1) (layers "*.Cu" "*.Mask")
+    (pad "9" thru_hole oval (at 0 10.16 180) (size 1.7 1.7) (drill 1) (layers "*.Cu" "*.Mask")
       (net 51 "/46") (pinfunction "Pin_9") (pintype "passive"))
-    (pad "10" thru_hole oval (at 2.54 10.16) (size 1.7 1.7) (drill 1) (layers "*.Cu" "*.Mask")
+    (pad "10" thru_hole oval (at 2.54 10.16 180) (size 1.7 1.7) (drill 1) (layers "*.Cu" "*.Mask")
       (net 52 "/47") (pinfunction "Pin_10") (pintype "passive"))
-    (pad "11" thru_hole oval (at 0 12.7) (size 1.7 1.7) (drill 1) (layers "*.Cu" "*.Mask")
+    (pad "11" thru_hole oval (at 0 12.7 180) (size 1.7 1.7) (drill 1) (layers "*.Cu" "*.Mask")
       (net 53 "/44") (pinfunction "Pin_11") (pintype "passive"))
-    (pad "12" thru_hole oval (at 2.54 12.7) (size 1.7 1.7) (drill 1) (layers "*.Cu" "*.Mask")
+    (pad "12" thru_hole oval (at 2.54 12.7 180) (size 1.7 1.7) (drill 1) (layers "*.Cu" "*.Mask")
       (net 54 "/45") (pinfunction "Pin_12") (pintype "passive"))
-    (pad "13" thru_hole oval (at 0 15.24) (size 1.7 1.7) (drill 1) (layers "*.Cu" "*.Mask")
+    (pad "13" thru_hole oval (at 0 15.24 180) (size 1.7 1.7) (drill 1) (layers "*.Cu" "*.Mask")
       (net 55 "/42") (pinfunction "Pin_13") (pintype "passive"))
-    (pad "14" thru_hole oval (at 2.54 15.24) (size 1.7 1.7) (drill 1) (layers "*.Cu" "*.Mask")
+    (pad "14" thru_hole oval (at 2.54 15.24 180) (size 1.7 1.7) (drill 1) (layers "*.Cu" "*.Mask")
       (net 56 "/43") (pinfunction "Pin_14") (pintype "passive"))
-    (pad "15" thru_hole oval (at 0 17.78) (size 1.7 1.7) (drill 1) (layers "*.Cu" "*.Mask")
+    (pad "15" thru_hole oval (at 0 17.78 180) (size 1.7 1.7) (drill 1) (layers "*.Cu" "*.Mask")
       (net 57 "/40") (pinfunction "Pin_15") (pintype "passive"))
-    (pad "16" thru_hole oval (at 2.54 17.78) (size 1.7 1.7) (drill 1) (layers "*.Cu" "*.Mask")
+    (pad "16" thru_hole oval (at 2.54 17.78 180) (size 1.7 1.7) (drill 1) (layers "*.Cu" "*.Mask")
       (net 58 "/41") (pinfunction "Pin_16") (pintype "passive"))
-    (pad "17" thru_hole oval (at 0 20.32) (size 1.7 1.7) (drill 1) (layers "*.Cu" "*.Mask")
+    (pad "17" thru_hole oval (at 0 20.32 180) (size 1.7 1.7) (drill 1) (layers "*.Cu" "*.Mask")
       (net 59 "/38") (pinfunction "Pin_17") (pintype "passive"))
-    (pad "18" thru_hole oval (at 2.54 20.32) (size 1.7 1.7) (drill 1) (layers "*.Cu" "*.Mask")
+    (pad "18" thru_hole oval (at 2.54 20.32 180) (size 1.7 1.7) (drill 1) (layers "*.Cu" "*.Mask")
       (net 60 "/39") (pinfunction "Pin_18") (pintype "passive"))
-    (pad "19" thru_hole oval (at 0 22.86) (size 1.7 1.7) (drill 1) (layers "*.Cu" "*.Mask")
+    (pad "19" thru_hole oval (at 0 22.86 180) (size 1.7 1.7) (drill 1) (layers "*.Cu" "*.Mask")
       (net 61 "/36") (pinfunction "Pin_19") (pintype "passive"))
-    (pad "20" thru_hole oval (at 2.54 22.86) (size 1.7 1.7) (drill 1) (layers "*.Cu" "*.Mask")
+    (pad "20" thru_hole oval (at 2.54 22.86 180) (size 1.7 1.7) (drill 1) (layers "*.Cu" "*.Mask")
       (net 62 "/37") (pinfunction "Pin_20") (pintype "passive"))
-    (pad "21" thru_hole oval (at 0 25.4) (size 1.7 1.7) (drill 1) (layers "*.Cu" "*.Mask")
+    (pad "21" thru_hole oval (at 0 25.4 180) (size 1.7 1.7) (drill 1) (layers "*.Cu" "*.Mask")
       (net 63 "/34") (pinfunction "Pin_21") (pintype "passive"))
-    (pad "22" thru_hole oval (at 2.54 25.4) (size 1.7 1.7) (drill 1) (layers "*.Cu" "*.Mask")
+    (pad "22" thru_hole oval (at 2.54 25.4 180) (size 1.7 1.7) (drill 1) (layers "*.Cu" "*.Mask")
       (net 64 "/35") (pinfunction "Pin_22") (pintype "passive"))
-    (pad "23" thru_hole oval (at 0 27.94) (size 1.7 1.7) (drill 1) (layers "*.Cu" "*.Mask")
+    (pad "23" thru_hole oval (at 0 27.94 180) (size 1.7 1.7) (drill 1) (layers "*.Cu" "*.Mask")
       (net 14 "/32") (pinfunction "Pin_23") (pintype "passive"))
-    (pad "24" thru_hole oval (at 2.54 27.94) (size 1.7 1.7) (drill 1) (layers "*.Cu" "*.Mask")
+    (pad "24" thru_hole oval (at 2.54 27.94 180) (size 1.7 1.7) (drill 1) (layers "*.Cu" "*.Mask")
       (net 65 "/33") (pinfunction "Pin_24") (pintype "passive"))
-    (pad "25" thru_hole oval (at 0 30.48) (size 1.7 1.7) (drill 1) (layers "*.Cu" "*.Mask")
+    (pad "25" thru_hole oval (at 0 30.48 180) (size 1.7 1.7) (drill 1) (layers "*.Cu" "*.Mask")
       (net 13 "/30") (pinfunction "Pin_25") (pintype "passive"))
-    (pad "26" thru_hole oval (at 2.54 30.48) (size 1.7 1.7) (drill 1) (layers "*.Cu" "*.Mask")
+    (pad "26" thru_hole oval (at 2.54 30.48 180) (size 1.7 1.7) (drill 1) (layers "*.Cu" "*.Mask")
       (net 66 "/31") (pinfunction "Pin_26") (pintype "passive"))
-    (pad "27" thru_hole oval (at 0 33.02) (size 1.7 1.7) (drill 1) (layers "*.Cu" "*.Mask")
+    (pad "27" thru_hole oval (at 0 33.02 180) (size 1.7 1.7) (drill 1) (layers "*.Cu" "*.Mask")
       (net 12 "/28") (pinfunction "Pin_27") (pintype "passive"))
-    (pad "28" thru_hole oval (at 2.54 33.02) (size 1.7 1.7) (drill 1) (layers "*.Cu" "*.Mask")
+    (pad "28" thru_hole oval (at 2.54 33.02 180) (size 1.7 1.7) (drill 1) (layers "*.Cu" "*.Mask")
       (net 67 "/29") (pinfunction "Pin_28") (pintype "passive"))
-    (pad "29" thru_hole oval (at 0 35.56) (size 1.7 1.7) (drill 1) (layers "*.Cu" "*.Mask")
+    (pad "29" thru_hole oval (at 0 35.56 180) (size 1.7 1.7) (drill 1) (layers "*.Cu" "*.Mask")
       (net 11 "/26") (pinfunction "Pin_29") (pintype "passive"))
-    (pad "30" thru_hole oval (at 2.54 35.56) (size 1.7 1.7) (drill 1) (layers "*.Cu" "*.Mask")
+    (pad "30" thru_hole oval (at 2.54 35.56 180) (size 1.7 1.7) (drill 1) (layers "*.Cu" "*.Mask")
       (net 68 "/27") (pinfunction "Pin_30") (pintype "passive"))
-    (pad "31" thru_hole oval (at 0 38.1) (size 1.7 1.7) (drill 1) (layers "*.Cu" "*.Mask")
+    (pad "31" thru_hole oval (at 0 38.1 180) (size 1.7 1.7) (drill 1) (layers "*.Cu" "*.Mask")
       (net 6 "/24") (pinfunction "Pin_31") (pintype "passive"))
-    (pad "32" thru_hole oval (at 2.54 38.1) (size 1.7 1.7) (drill 1) (layers "*.Cu" "*.Mask")
+    (pad "32" thru_hole oval (at 2.54 38.1 180) (size 1.7 1.7) (drill 1) (layers "*.Cu" "*.Mask")
       (net 69 "/25") (pinfunction "Pin_32") (pintype "passive"))
-    (pad "33" thru_hole oval (at 0 40.64) (size 1.7 1.7) (drill 1) (layers "*.Cu" "*.Mask")
+    (pad "33" thru_hole oval (at 0 40.64 180) (size 1.7 1.7) (drill 1) (layers "*.Cu" "*.Mask")
       (net 5 "/22") (pinfunction "Pin_33") (pintype "passive"))
-    (pad "34" thru_hole oval (at 2.54 40.64) (size 1.7 1.7) (drill 1) (layers "*.Cu" "*.Mask")
+    (pad "34" thru_hole oval (at 2.54 40.64 180) (size 1.7 1.7) (drill 1) (layers "*.Cu" "*.Mask")
       (net 70 "/23") (pinfunction "Pin_34") (pintype "passive"))
-    (pad "35" thru_hole oval (at 0 43.18) (size 1.7 1.7) (drill 1) (layers "*.Cu" "*.Mask")
+    (pad "35" thru_hole oval (at 0 43.18 180) (size 1.7 1.7) (drill 1) (layers "*.Cu" "*.Mask")
       (net 27 "+5V") (pinfunction "Pin_35") (pintype "passive"))
-    (pad "36" thru_hole oval (at 2.54 43.18) (size 1.7 1.7) (drill 1) (layers "*.Cu" "*.Mask")
+    (pad "36" thru_hole oval (at 2.54 43.18 180) (size 1.7 1.7) (drill 1) (layers "*.Cu" "*.Mask")
       (net 27 "+5V") (pinfunction "Pin_36") (pintype "passive"))
     (model "${KICAD6_3DMODEL_DIR}/Connector_PinHeader_2.54mm.3dshapes/PinHeader_2x18_P2.54mm_Vertical.wrl"
